File: pcb/PaprControlPCB/Papra v0.3.sch (EAGLE design)
At the start: 33 parts, among them Q1 AO3400A (C20917), U1 LP2985-50DBVR (C74511), U2 ATTINYX04SOIC14

Commit message: v0.3 release candidate
Connections:
- net +5V: now also POT1.3; no longer POT1.1
- net FAN-PWM: now also U2.PB0/AIN11/XDIR/SCL/WO0; no longer U2.PA3/EXTCLK/AIN3/XCK(ALT)/SCK/WO3
- net FAN-SENSE: now also U2.PA3/EXTCLK/AIN3/XCK(ALT)/SCK/WO3; no longer U2.PB1/AIN10/XCK/SDA/WO1
- net GND: now also POT1.1; no longer POT1.3
- net LED4: now also U2.PB1/AIN10/XCK/SDA/WO1; no longer U2.PB0/AIN11/XDIR/SCL/WO0
Changed lines of the file:
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@@
    - 12V LED (was 1K1, is 1K2)
 v.3
-- Added 1A Resettable Fuse to 12V</text>
+- Added 1A Resettable Fuse to 12V
+- Moved FAN-PWM to WO0 (was WO3)
+- Flipped Potentiometer 5V &amp; GND
+</text>
 </plain>
 <instances>
@@
 <attribute name="VALUE" x="142.24" y="101.6" size="1.778" layer="96" rot="MR90"/>
 </instance>
-<instance part="GND6" gate="1" x="139.7" y="88.9" smashed="yes">
-<attribute name="VALUE" x="137.16" y="86.36" size="1.778" layer="96"/>
+<instance part="GND6" gate="1" x="132.08" y="116.84" smashed="yes">
+<attribute name="VALUE" x="129.54" y="114.3" size="1.778" layer="96"/>
 </instance>
 <instance part="H4" gate="G$1" x="91.44" y="104.14" smashed="yes" rot="MR0">
@@
 <attribute name="VALUE" x="15.24" y="200.66" size="1.778" layer="96" rot="R90"/>
 </instance>
-<instance part="P+9" gate="1" x="139.7" y="121.92" smashed="yes">
-<attribute name="VALUE" x="137.16" y="116.84" size="1.778" layer="96" rot="R90"/>
+<instance part="P+9" gate="1" x="132.08" y="93.98" smashed="yes">
+<attribute name="VALUE" x="129.54" y="88.9" size="1.778" layer="96" rot="R90"/>
 </instance>
 <instance part="R2" gate="G$1" x="114.3" y="40.64" smashed="yes" rot="R90">
@@
 </segment>
 <segment>
-<pinref part="POT1" gate="G$1" pin="3"/>
-<pinref part="GND6" gate="1" pin="GND"/>
-<wire x1="139.7" y1="91.44" x2="139.7" y2="96.52" width="0.1524" layer="91"/>
-</segment>
-<segment>
 <pinref part="R10" gate="G$1" pin="2"/>
 <pinref part="GND9" gate="1" pin="GND"/>
 <wire x1="180.34" y1="78.74" x2="177.8" y2="78.74" width="0.1524" layer="91"/>
+</segment>
+<segment>
+<pinref part="GND6" gate="1" pin="GND"/>
+<wire x1="132.08" y1="119.38" x2="132.08" y2="124.46" width="0.1524" layer="91"/>
+<pinref part="POT1" gate="G$1" pin="1"/>
+<wire x1="132.08" y1="124.46" x2="139.7" y2="124.46" width="0.1524" layer="91"/>
+<wire x1="139.7" y1="124.46" x2="139.7" y2="111.76" width="0.1524" layer="91"/>
 </segment>
 </net>
@@
 </segment>
 <segment>
-<pinref part="POT1" gate="G$1" pin="1"/>
 <pinref part="P+9" gate="1" pin="+5V"/>
-<wire x1="139.7" y1="119.38" x2="139.7" y2="111.76" width="0.1524" layer="91"/>
+<wire x1="132.08" y1="91.44" x2="132.08" y2="86.36" width="0.1524" layer="91"/>
+<pinref part="POT1" gate="G$1" pin="3"/>
+<wire x1="132.08" y1="86.36" x2="139.7" y2="86.36" width="0.1524" layer="91"/>
+<wire x1="139.7" y1="86.36" x2="139.7" y2="96.52" width="0.1524" layer="91"/>
 </segment>
 </net>
@@
 </segment>
 <segment>
-<pinref part="POT1" gate="G$1" pin="5"/>
-<pinref part="P+1" gate="1" pin="+12V"/>
-<wire x1="152.4" y1="119.38" x2="152.4" y2="109.22" width="0.1524" layer="91"/>
-</segment>
-<segment>
 <pinref part="P+4" gate="1" pin="+12V"/>
 <pinref part="F1" gate="G$1" pin="2"/>
 <wire x1="208.28" y1="195.58" x2="208.28" y2="193.04" width="0.1524" layer="91"/>
+</segment>
+<segment>
+<pinref part="POT1" gate="G$1" pin="5"/>
+<pinref part="P+1" gate="1" pin="+12V"/>
+<wire x1="152.4" y1="109.22" x2="152.4" y2="119.38" width="0.1524" layer="91"/>
 </segment>
 </net>
@@
 </segment>
 <segment>
-<wire x1="78.74" y1="182.88" x2="111.76" y2="182.88" width="0.1524" layer="91"/>
-<label x="81.28" y="182.88" size="1.778" layer="95"/>
-<pinref part="U2" gate="G$1" pin="PA3/EXTCLK/AIN3/XCK(ALT)/SCK/WO3"/>
+<pinref part="U2" gate="G$1" pin="PB0/AIN11/XDIR/SCL/WO0"/>
+<wire x1="78.74" y1="162.56" x2="111.76" y2="162.56" width="0.1524" layer="91"/>
+<label x="81.28" y="162.56" size="1.778" layer="95"/>
 </segment>
 </net>
@@
 <wire x1="152.4" y1="93.98" x2="170.18" y2="93.98" width="0.1524" layer="91"/>
 <label x="160.02" y="93.98" size="1.778" layer="95"/>
-<pinref part="POT1" gate="G$1" pin="4"/>
-<wire x1="152.4" y1="99.06" x2="152.4" y2="93.98" width="0.1524" layer="91" style="longdash"/>
 <pinref part="LED5" gate="G$1" pin="A"/>
 <wire x1="157.48" y1="78.74" x2="152.4" y2="78.74" width="0.1524" layer="91"/>
 <wire x1="152.4" y1="78.74" x2="152.4" y2="93.98" width="0.1524" layer="91"/>
+<pinref part="POT1" gate="G$1" pin="4"/>
+<wire x1="152.4" y1="93.98" x2="152.4" y2="99.06" width="0.1524" layer="91"/>
 <junction x="152.4" y="93.98"/>
 </segment>
@@
 <net name="LED4" class="0">
 <segment>
-<pinref part="U2" gate="G$1" pin="PB0/AIN11/XDIR/SCL/WO0"/>
-<wire x1="78.74" y1="162.56" x2="111.76" y2="162.56" width="0.1524" layer="91"/>
-<label x="81.28" y="162.56" size="1.778" layer="95"/>
-</segment>
-<segment>
 <label x="66.04" y="22.86" size="1.778" layer="95"/>
 <wire x1="50.8" y1="22.86" x2="76.2" y2="22.86" width="0.1524" layer="91"/>
 <pinref part="R7" gate="G$1" pin="2"/>
 </segment>
+<segment>
+<pinref part="U2" gate="G$1" pin="PB1/AIN10/XCK/SDA/WO1"/>
+<wire x1="78.74" y1="165.1" x2="111.76" y2="165.1" width="0.1524" layer="91"/>
+<label x="81.28" y="165.1" size="1.778" layer="95"/>
+</segment>
 </net>
 <net name="LED1-R" class="0">
@@
 </segment>
 <segment>
-<pinref part="U2" gate="G$1" pin="PB1/AIN10/XCK/SDA/WO1"/>
-<wire x1="78.74" y1="165.1" x2="111.76" y2="165.1" width="0.1524" layer="91"/>
-<label x="81.28" y="165.1" size="1.778" layer="95"/>
-</segment>
-</net>
+<wire x1="78.74" y1="182.88" x2="111.76" y2="182.88" width="0.1524" layer="91"/>
+<label x="81.28" y="182.88" size="1.778" layer="95"/>
+<pinref part="U2" gate="G$1" pin="PA3/EXTCLK/AIN3/XCK(ALT)/SCK/WO3"/>
+</segment>
+</net>
