File: pcb/PaprControlPCB/PCB Design Files/Papra v0.5.brd (EAGLE design)
At the start: 32 x 45 mm, 33 parts, among them Q1 AO3400A (C20917), U1 LP2985-50DBVR (C74511), U2 ATTINYX04SOIC14

Commit message: V.5 Release candidate
Parts:
- added D2, D3: MBR2H100SFT3G C96515, Diode:SODFL3718X115
- added F2: 13.2V 1.8A (C70081), SparkFun-Fuses:1206
- added Q2: AO3400A (C20917), Transistor:SOT23
- added R12: 10K 0805W8F1002T5E (C17414), rcl:R0805
- added R13: 120 0805W8F1200T5E (C17437), rcl:R0805
- added SG1: YS-MBZ12095DYB12 C409840, buzzer:F/TMB
- D1: value SS34 (C8678) -> MBR2H100SFT3G C96515; device Diode:DIOM5226X290N -> Diode:SODFL3718X115
- LED1, LED2, LED3, LED4: value NCD0805R1 (C84256) -> NCD0805G1 C84260
- R3: value 4.7K 0805W8F4701T5E (C17673) -> 1K2 0805W8F1201T5E (C17379)
- R4, R5, R6, R7: value 330 0805W8F3300T5E (C17630) -> 120 0805W8F1200T5E (C17437)
- R8: value 47R 0805W8F470JT5E (C17714) -> 120 0805W8F1200T5E (C17437)
- moved R3 17.8 mm to (-9.30, 16.0), turned to 270 degrees
- moved C4 12.5 mm to (5.59, 5.59), turned to 180 degrees
- moved R8 11.8 mm to (10.9, -3.81), turned to 270 degrees
- moved R9 10.0 mm to (8.76, -3.81), turned to 270 degrees
- moved H3 9.29 mm to (17.4, 20.0), turned to 180 degrees
- moved Q1 8.75 mm to (14.7, -5.33), turned to 180 degrees
- moved R2 6.33 mm to (12.2, 16.5)
- moved R1 6.27 mm to (9.91, 16.5)
- moved D1 4.57 mm to (11.2, -7.62), turned to 0 degrees
- moved F1 2.34 mm to (5.59, 7.87), turned to 180 degrees
Connections:
- net FAN-SENSE renamed UNUSED
- removed net 12V-F: BATT+.1, BATT+.2, F1.1, H1.PWR
- new net 12V-BAT: BATT+.1, BATT+.2, D2.2
- new net 12V-DC: D3.2, H1.PWR
- new net 12V-DIODEOR: D2.1, D3.1, F1.1, F2.1
- new net 12V-FAN: D1.1, F2.2, H2.SIGNAL
- new net BUZZER: R12.2, R13.2, U2.8
- new net BUZZER-GND: Q2.3, SG1.-
- new net FETGATE1: Q2.1, R13.1
- new net PINS: H2.P$1, H2.P$2
- net +12V: now also SG1.+; no longer D1.1, H2.SIGNAL
- net GND: now also Q2.2, R12.1
- net GND-SWITCH: no longer U2.2
- net LED4: now also U2.2; no longer U2.8
Routing:
- net 12V-FAN: track 0.00 -> 39.8 mm
- net BUZZER: track 0.00 -> 38.3 mm, vias 0 -> 2
- net UPDI: track 46.3 -> 9.30 mm, vias 0 -> 1
- net UPDI/RST: track 13.6 -> 41.0 mm, vias 0 -> 3
- net 12V-F: track 24.7 -> 0.00 mm
- net +12V: track 93.5 -> 113.9 mm, vias 2 -> 0
- net GND: track 48.3 -> 67.1 mm
- net 12V-BAT: track 0.00 -> 18.6 mm
- net GND-SWITCH: track 41.0 -> 22.9 mm, vias 1 -> 0
- net FAN-PWM: track 21.6 -> 6.93 mm, vias 2 -> 0
- net FAN-GND: track 19.8 -> 6.05 mm
- net BUZZER-GND: track 0.00 -> 12.3 mm
- net EXPANSIONTX: track 37.2 -> 49.2 mm, vias 2 -> 1
- net ADC-BAT: track 19.2 -> 31.0 mm
- net PINS: track 0.00 -> 10.2 mm
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Other:
- board size 32 x 45 mm -> 36 x 45 mm
- board text added: "26APR2021"
- board text added: "PA3"
- board text added: "PAPRA V0.5"
- board text added: "UPDI R"
- board text removed: "22MAR2021"
- board text removed: "PAPRA V0.4"
