File: pcb/PaprControlPCB/PCB Design Files/Papra v0.5.sch (EAGLE design)
At the start: 33 parts, among them Q1 AO3400A (C20917), U1 LP2985-50DBVR (C74511), U2 ATTINYX04SOIC14

Commit message: V.5 Release candidate
Parts:
- added D2, D3: MBR2H100SFT3G C96515, Diode:DIODE_DO-219-AB(SOD123F)
- added F2: 13.2V 1.8A (C70081), SparkFun-Fuses:PPTC_HALF-AMP
- added Q2: AO3400A (C20917), Transistor:NMOSFET_BSS123-SOT23
- added R12: 10K 0805W8F1002T5E (C17414), rcl:R-US_R0805
- added R13: 120 0805W8F1200T5E (C17437), rcl:R-US_R0805
- added SG1: YS-MBZ12095DYB12 C409840, buzzer:F/TMB
- D1: value SS34 (C8678) -> MBR2H100SFT3G C96515; device Diode:DIODEDO-214AC(SMA) -> Diode:DIODE_DO-219-AB(SOD123F)
- LED1, LED2, LED3, LED4: value NCD0805R1 (C84256) -> NCD0805G1 C84260
- R3: value 4.7K 0805W8F4701T5E (C17673) -> 1K2 0805W8F1201T5E (C17379)
- R4, R5, R6, R7: value 330 0805W8F3300T5E (C17630) -> 120 0805W8F1200T5E (C17437)
- R8: value 47R 0805W8F470JT5E (C17714) -> 120 0805W8F1200T5E (C17437)
Connections:
- net FAN-SENSE renamed UNUSED
- removed net 12V-F: BATT+.PIN@1, BATT+.PIN@2, F1.1, H1.TIP
- new net 12V-BAT: BATT+.PIN@1, BATT+.PIN@2, D2.A
- new net 12V-DC: D3.A, H1.TIP
- new net 12V-DIODEOR: D2.C, D3.C, F1.1, F2.1
- new net 12V-FAN: D1.C, F2.2, H2.P1
- new net BUZZER: R12.2, R13.2, U2.PB1/AIN10/XCK/SDA/WO1
- new net BUZZER-GND: Q2.D, SG1.-
- new net FETGATE1: Q2.G, R13.1
- new net PINS: H2.P3
- net +12V: now also SG1.+; no longer D1.C, H2.P1
- net GND: now also Q2.S, R12.1
- net GND-SWITCH: no longer U2.PA4/AIN4/XDIR(ALT)/SS/WO4/LUT-OUT0
- net LED4: now also U2.PA4/AIN4/XDIR(ALT)/SS/WO4/LUT-OUT0; no longer U2.PB1/AIN10/XCK/SDA/WO1
Other:
- note added: "BUZZER"
- moved on the sheet: C1, C4, D1, F1, LED5, POT1, Q1, R10, R11, R8, R9
