File: pcb/PaprControlPCB/PCB Design Files/Papra v0.6.sch (EAGLE design)
At the start: 40 parts, among them Q1 AO3400A (C20917), Q2 AO3400A (C20917), U1 LP2985-50DBVR (C74511), U2 ATTINYX04SOIC14

Commit message: Board ready for review
Closes #53
Parts:
- removed D2, D3: MBR2H100SFT3G C96515, Diode:DIODE_DO-219-AB(SOD123F)
- removed F1, F2: 13.2V 1.8A (C70081), SparkFun-Fuses:PPTC_HALF-AMP
- removed H3: 1X4-BIG, adafruit:1X4-BIG
- removed R3: 1K2 0805W8F1201T5E (C17379), rcl:R-US_R0805
- added B2: PTR1PAD1-13, testpad:PTR1PAD1-13
- added C5: 3.6nF, rcl:C-USC0805
- added C6: 2.7nF, rcl:C-USC0805
- added C7, C8: 1uF CL21B105KBFNNNE (C28323), rcl:C-USC0805
- added C9: .1uF CL21B104KBFNNNE (C49678 ), rcl:C-USC0805
- added R14: 470K, rcl:R-US_R0805
- added R15: 82K, rcl:R-US_R0805
- added R16: 390K, rcl:R-US_R0805
- added R17: 1K, rcl:R-US_R0805
- added R18: 360K, rcl:R-US_R0805
- added R19: 56K, rcl:R-US_R0805
- added R20: 10K 0805W8F1002T5E (C17414), rcl:R-US_R0805
- added U9: TPS259472ARPWR, TI e-Fuse:TPS259472ARPWR
- LED1, LED2, LED3, LED4: value NCD0805G1 C84260 -> NCD0603G1 C84267
- Q1, Q2: value AO3400A (C20917) -> BSS123
Connections:
- removed net 12V-BAT: BATT+.PIN@1, BATT+.PIN@2, D2.A
- removed net 12V-DC: D3.A, H1.TIP
- removed net 12V-DIODEOR: D2.C, D3.C, F1.1, F2.1
- removed net 12V-FAN: D1.C, F2.2, H2.P1
- removed net EXPANSIONRX: H3.3, U2.PB3/RXD/WO0(ALT)
- removed net EXPANSIONTX: H3.2, U2.PB2/EVOUT1/TXD/WO2
- removed net UNUSED: U2.PA3/EXTCLK/AIN3/XCK(ALT)/SCK/WO3
- removed net UPDI/RST: R3.1, U2.PA0/RESET/UPDI/AIN0/LUT0-IN0
- new net 12V-IN: BATT+.PIN@1, BATT+.PIN@2, C9.1, H1.TIP, R14.2, U9.IN
- new net DEBUGTX: B2.TP, U2.PB2/EVOUT1/TXD/WO2
- new net DVDT: C5.1, U9.DVDT
- new net EN/UVLO: R14.1, R15.2, U9.EN/UVLO
- new net ILM: R17.2, U2.PA1/AIN1/TXD(ALT)/MOSI/LUTO-IN1, U9.ILM
- new net ITIMER: C6.1, U9.ITIMER
- new net OVCSEL: R16.2, U9.OVCSEL
- new net PG: R20.1, U2.PB3/RXD/WO0(ALT), U9.PG
- new net PGTH: R18.1, R19.2, U9.PGTH
- net +12V: now also C7.1, D1.C, H2.P1, R18.2, U9.OUT; no longer F1.2, H3.4
- net +5V: now also C8.1, R20.2
- net ADC-BAT: now also U2.PA3/EXTCLK/AIN3/XCK(ALT)/SCK/WO3; no longer U2.PA1/AIN1/TXD(ALT)/MOSI/LUTO-IN1
- net GND: now also C5.2, C6.2, C7.2, C8.2, C9.2, R15.1, R16.1, R17.1, R19.1, U9.GND; no longer H3.1
- net LED1: now also U2.PA4/AIN4/XDIR(ALT)/!SS!/WO4/LUT-OUT0; no longer U2.PA5/AIN5/OUT/WO5/WO
- net LED2: now also U2.PA5/AIN5/OUT/WO5/WO; no longer U2.PA6/AIN6/AINNO0/MOSI(ALT)
- net LED3: now also U2.PA6/AIN6/AINNO0/MOSI(ALT); no longer U2.PA7/AIN7/AINP0/MISO(ALT)/LUT1-OUT
- net LED4: now also U2.PA7/AIN7/AINP0/MISO(ALT)/LUT1-OUT; no longer U2.PA4/AIN4/XDIR(ALT)/SS/WO4/LUT-OUT0
- net UPDI: now also U2.PA0/!RESET!/UPDI/AIN0/LUT0-IN0; no longer R3.2
Other:
- note added: "DigiKey Buzzer Option https://www.digikey.com/en/products/detail/cui-devices/CMI-1210-92T/13245502"
- note added: "E-FUSE"
- note added: "R & C values TBD"
- note added: "maximum amperage DC Jack - 5A Fan Fet - 5.7A"
- note added: "maximum input voltage Resistor Divider - 14V Buzzer - 15V Regulator - 16V C4 - 16V Fan Fet - 30V C1 - 50V"
- note removed: "EXPANSION"
- moved on the sheet: BATT+, BATT-, C1, C2, C3, C4, D1, H1, H2, LED1, LED2, LED3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

Commit message: Updates based on feedback
Parts:
- R15: value 82K -> 75K
Other:
- note added: "R & C values to be tested"
- note removed: "R & C values TBD"
Changed lines of the file:
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@@
 <part name="U9" library="TI e-Fuse" deviceset="TPS259472ARPWR" device="" package3d_urn="urn:adsk.eagle:package:30039395/1"/>
 <part name="R14" library="rcl" library_urn="urn:adsk.eagle:library:334" deviceset="R-US_" device="R0805" package3d_urn="urn:adsk.eagle:package:23553/2" value="470K"/>
-<part name="R15" library="rcl" library_urn="urn:adsk.eagle:library:334" deviceset="R-US_" device="R0805" package3d_urn="urn:adsk.eagle:package:23553/2" value="82K"/>
+<part name="R15" library="rcl" library_urn="urn:adsk.eagle:library:334" deviceset="R-US_" device="R0805" package3d_urn="urn:adsk.eagle:package:23553/2" value="75K"/>
 <part name="GND11" library="supply1" library_urn="urn:adsk.eagle:library:371" deviceset="GND" device=""/>
 <part name="R16" library="rcl" library_urn="urn:adsk.eagle:library:334" deviceset="R-US_" device="R0805" package3d_urn="urn:adsk.eagle:package:23553/2" value="390K"/>
@@
 v0.6
 - Replaced reverse polarity diode and fuses with E-FUSE circuit
-- Connected PowerGood to ATtiny
+- Connected PowerGood &amp; ILM to ATtiny
 - Added 0.1uF to ATtiny
 - Removed expansion header
 - Connected TXD to touchpad for debug
-- Connected ATtiny to PG
 - Moved ADC-BAT to pin 13
-- Renumbered LED1-4 on ATtiny
+- Renumbered LED1-4 on ATtiny for easy routing
 </text>
 <text x="93.98" y="111.76" size="1.778" layer="91">BUZZER</text>
@@
 https://www.digikey.com/en/products/detail/cui-devices/CMI-1210-92T/13245502</text>
 <text x="218.44" y="111.76" size="1.778" layer="91">DC POWER INPUTS</text>
-<text x="200.66" y="170.18" size="3.81" layer="91">R &amp; C values TBD</text>
+<text x="205.74" y="165.1" size="3.81" layer="91">R &amp; C values
+to be tested</text>
 </plain>
 <instances>
