File: pcb/PaprControlPCB/PCB Design Files/Papra v0.7.sch (EAGLE design)
At the start: 48 parts, among them Q1 BSS123, Q2 BSS123, U1 LP2985-50DBVR (C74511), U2 ATTINYX04SOIC14, U9 TPS259472ARPWR

Commit message: Updating to v0.7
Closes #59
Parts:
- removed B2: PTR1PAD1-13, testpad:PTR1PAD1-13
- added +12V: PTR1B1,27, testpad:PTR1B1,27
- added C10: .1uF CL21B104KBFNNNE (C49678 ), rcl:C-USC0805
- added C11: 1uF CL21B105KBFNNNE (C28323), rcl:C-USC0805
- added C12: 220uF, rcl:CPOL-USF
- added D2: MBR2H100SFT3G C96515, Diode:DIODE_DO-219-AB(SOD123F)
- added TX: PTR1PAD1-13, testpad:PTR1PAD1-13
- C7: value 1uF CL21B105KBFNNNE (C28323) -> 10uF
Connections:
- removed net PINS: H2.P3
- net +12V: now also +12V.TP, C12.+, D2.C
- net 12V-IN: now also C11.1
- net DEBUGTX: now also TX.TP; no longer B2.TP
- net EN/UVLO: now also C10.1
- net GND: now also C10.2, C11.2, C12.-, D2.A
Other:
- moved on the sheet: C1, C3, C4, C5, C6, C7, C9, R11, R14, R15, R16, R17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
