File: pcb/PaprControlPCB/PCB Design Files/Papra v0.7.2.brd (EAGLE design)
At the start: 39 x 45 mm, 53 parts, among them Q1 BSS123, Q2 BSS123, U1 LP2985-50DBVR (C74511), U2 ATTINYX04SOIC14, U9 TPS259472ARPWR

Commit message: DFM Update
Closes #72
Closes #73
Closes #74
Routing:
- net +5V: track 92.1 -> 90.9 mm
Other:
- board text added: "02FEB2023"
- board text added: "5V"
- board text added: "C:/Users/pc/OneDrive/GitHub/PrivateEagle/projects/Papr/oshw_cert_us002161 bw.bmp"
- board text added: "Changelog v0.2 - BATTERY Tabs swapped (polarity, same position) - SMT Components Moved, won't affect mechanical - D1 package changed (was SMB, is SMA) v0.3 changelog (see schematic for signal changes) - Added mounting hole - Added fuse, moved SMT components to fit - Adjustments for JLC DRU, pad override was 40%, reduced to 25% - Silk cleanup - Changed Battery Tab package to round pads (was square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"
- board text added: "GND"
- board text added: "PAPRA V0.7.2"
- board text removed: "05JAN2022"
- board text removed: "PAPRA V0.7"
- board text removed: "v.2 changelog - BATTERY Tabs swapped (polarity, same position) - SMT Components Moved, won't affect mechanical - D1 package changed (was SMB, is SMA) v.3 changelog (see schematic for signal changes) - Added mounting hole - Added fuse, moved SMT components to fit - Adjustments for JLC DRU, pad override was 40%, reduced to 25% - Silk cleanup - Changed Battery Tab package to round pads (was square) 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"
