File: components/a-tet-001113/components/p-tet-000166/src/Papra TH_eagle.brd (EAGLE design)
At the start: 45 x 65.5 mm, 37 parts, among them Q1 P-FET, Q2 N-FET, Q3 N-FET, U1 QT Py ESP32-S3

Commit message: Ready for production - adding gerbers and final PCB design files
Parts:
- moved R10 0.25 mm to (-8.75, -21.6)
- moved R7 0.25 mm to (-8.78, -12.1)
- moved R8 0.25 mm to (-8.78, -15.2)
- moved R9 0.25 mm to (-8.78, -18.4)
Routing:
- net FAN-PWM: track 43.1 -> 42.0 mm
- net 12V-SWITCHED: track 53.6 -> 53.0 mm
- net BUZZER: track 70.7 -> 70.1 mm
Other:
- board text added: "PAPRA TH V1.0.0 PCB: P-TET-000166 PCBA: A-TET-001113 08MAR2023"
- board text added: "https://github.com/tetrabiodistributed/papra-pcba"
- board text added: "info@tetrab.io"
- board text removed: "07MAR2023"
- board text removed: "C:/Users/pc/Downloads/Tetra Logo Package/tetra.bmp"
- board text removed: "C:/Users/pc/OneDrive/GitHub/PrivateEagle/projects/Papr/oshw_cert_us002161 bw.bmp"
